Commit message: 修bug

File: 大作业/percep_node+track/right_angle_stack/urdf/right_angle_car.urdf.xacro (robot description, xacro)
@@ -1,5 +1,4 @@
 <?xml version="1.0"?>
 <robot name="right_angle_car" xmlns:xacro="http://www.ros.org/wiki/xacro">
-  <xacro:property name="pi" value="3.141592653589793"/>
   <xacro:property name="wheel_radius" value="0.18"/>
   <xacro:property name="wheel_width" value="0.08"/>
